Commit message: Castor wheel

File: description/robot_core.xacro (robot description, xacro)
@@ -11,5 +11,5 @@
     </material>
     <material name="black">
-        <color rgba="0.0 0.0 0.0 0.0"/>
+        <color rgba="0.0 0.0 0.0 1.0"/>
     </material>
     <link name="base_link">
@@ -17,14 +17,55 @@
     <joint name="chassis_joint" type="fixed">
         <parent link="base_link"/>
-        <child link="chassis_link"/>
+        <child link="chassis"/>
         <origin xyz="-0.1 0.0 0.0"/>
     </joint>
-    <link name="chassis_link">
+    <link name="chassis">
         <visual>
+            <origin xyz="0.15 0.0 0.075"/>
             <geometry>
                 <box size="0.3 0.3 0.15"/>
             </geometry>
-            <material name="white">
-            </material>
+            <material name="white"/>
+        </visual>
+    </link>
+    <joint name="left_wheel_joint" type="continuous">
+        <parent link="base_link"/>
+        <child link="left_wheel"/>
+        <origin xyz="0.0 0.175 0.0" rpy="-${pi/2} 0.0 0.0"/>
+        <axis xyz="0.0 0.0 1.0"/>
+    </joint>
+    <link name="left_wheel">
+        <visual>
+            <geometry>
+                <cylinder radius="0.05" length="0.04"/>
+            </geometry>
+            <material name="blue"/>
+        </visual>
+    </link>
+    <joint name="right_wheel_joint" type="continuous">
+        <parent link="base_link"/>
+        <child link="right_wheel"/>
+        <origin xyz="0.0 -0.175 0.0" rpy="${pi/2} 0.0 0.0"/>
+        <axis xyz="0.0 0.0 -1.0"/>
+    </joint>
+    <link name="right_wheel">
+        <visual>
+            <geometry>
+                <cylinder radius="0.05" length="0.04"/>
+            </geometry>
+            <material name="blue"/>
+        </visual>
+    </link>
+    <joint name="caster_wheel_joint" type="fixed">
+        <parent link="chassis"/>
+        <child link="caster_wheel"/>
+        <origin xyz="0.24 0.0 0.0"/>
+    </joint>
+    <link name="caster_wheel">
+        <visual>
+            <geometry>
+                <sphere radius="0.05"/>
+            </geometry>
+            <material name="black"/>
         </visual>
     </link>

Commit message: Add inertial macros

File: description/robot_core.xacro (robot description, xacro)
@@ -1,4 +1,5 @@
 <?xml version="1.0"?>
 <robot xmlns:xacro="http://www.ros.org/wiki/xacro">
+    <xacro:include filename="inertial_macros.xacro"/>
     <material name="white">
         <color rgba="1.0 1.0 1.0 1.0"/>
@@ -28,4 +29,11 @@
             <material name="white"/>
         </visual>
+        <collision>
+            <origin xyz="0.15 0.0 0.075"/>
+            <geometry>
+                <box size="0.3 0.3 0.15"/>
+            </geometry>
+            <material name="white"/>
+        </collision>
     </link>
     <joint name="left_wheel_joint" type="continuous">
@@ -42,4 +50,10 @@
             <material name="blue"/>
         </visual>
+        <collision>
+            <geometry>
+                <cylinder radius="0.05" length="0.04"/>
+            </geometry>
+            <material name="blue"/>
+        </collision>
     </link>
     <joint name="right_wheel_joint" type="continuous">
@@ -56,4 +70,10 @@
             <material name="blue"/>
         </visual>
+        <collision>
+            <geometry>
+                <cylinder radius="0.05" length="0.04"/>
+            </geometry>
+            <material name="blue"/>
+        </collision>
     </link>
     <joint name="caster_wheel_joint" type="fixed">
@@ -69,4 +89,10 @@
             <material name="black"/>
         </visual>
+        <collision>
+            <geometry>
+                <sphere radius="0.05"/>
+            </geometry>
+            <material name="black"/>
+        </collision>
     </link>
 </robot>

Commit message: interial added

File: description/robot_core.xacro (robot description, xacro)
@@ -36,4 +36,7 @@
             <material name="white"/>
         </collision>
+        <xacro:inertial_box mass="0.5" x="0.3" y="0.3" z="0.15">
+            <origin xyz="0.15 0.0 0.75" rpy="0.0 0.0 0.0"/>
+        </xacro:inertial_box>
     </link>
     <joint name="left_wheel_joint" type="continuous">
@@ -56,4 +59,7 @@
             <material name="blue"/>
         </collision>
+        <xacro:inertial_sphere mass="0.1" radius="0.05">
+            <origin xyz="0.0 0.0 0.0" rpy="0.0 0.0 0.0"/>
+        </xacro:inertial_sphere>
     </link>
     <joint name="right_wheel_joint" type="continuous">
@@ -76,5 +82,8 @@
             <material name="blue"/>
         </collision>
-    </link>
+        <xacro:inertial_sphere mass="0.1" radius="0.05">
+            <origin xyz="0.0 0.0 0.0" rpy="0.0 0.0 0.0"/>
+        </xacro:inertial_sphere>
+     </link>
     <joint name="caster_wheel_joint" type="fixed">
         <parent link="chassis"/>

Commit message: Gazebo colours

File: description/robot_core.xacro (robot description, xacro)
@@ -40,4 +40,7 @@
         </xacro:inertial_box>
     </link>
+    <gazebo reference="chassis">
+        <material>Gazebo/White</material>
+    </gazebo>
     <joint name="left_wheel_joint" type="continuous">
         <parent link="base_link"/>
@@ -63,4 +66,7 @@
         </xacro:inertial_sphere>
     </link>
+    <gazebo reference="left_wheel">
+        <material>Gazebo/Blue</material>
+    </gazebo>
     <joint name="right_wheel_joint" type="continuous">
         <parent link="base_link"/>
@@ -86,4 +92,7 @@
         </xacro:inertial_sphere>
      </link>
+    <gazebo reference="right_wheel">
+        <material>Gazebo/Blue</material>
+    </gazebo>
     <joint name="caster_wheel_joint" type="fixed">
         <parent link="chassis"/>
@@ -105,3 +114,6 @@
         </collision>
     </link>
+    <gazebo reference="caster_wheel">
+        <material>Gazebo/Black</material>
+    </gazebo>
 </robot>
